File: Eagle/StandalonePRG.sch (EAGLE design)
At the start: 9 parts, among them J1 AVR_SPI_PRG_6PTH, J2 USB-B, Y1 16MHZ

Commit message: Example PCB
Parts:
- added C2: 4.7uF, SparkFun-Capacitors:4.7UF-6.3V-10%(0603)0603
- added D1, D2: (no value), SparkFun-LED:LED0603
- added R3: 300, SparkFun-Resistors:300OHM-1/10W-1%(0603)
- added S1: TAC_SWITCHSMD, SparkFun-Retired:TAC_SWITCHSMD
Connections:
- removed net N$26: U$1.PF7(ADC7)
- new net CLOCK: U$1.PB5(ADC12)
- new net LED: D2.A, U$1.PF7(ADC7)
- new net LGND: D1.C, D2.C, R3.2
- net BUTTON: now also S1.1
- net GND: now also C2.1, R3.1, S1.3
- net OSCK: no longer U$1.PB5(ADC12)
- net VCC: now also C2.2, D1.A
Changed lines of the file:
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@@
 <part name="J2" library="SparkFun-Connectors" deviceset="USB" device="PTH" value="USB-B"/>
 <part name="F1" library="SparkFun-PowerIC" deviceset="PTC" device="0603"/>
+<part name="S1" library="SparkFun-Retired" deviceset="TAC_SWITCH" device="SMD" value="TAC_SWITCHSMD"/>
+<part name="D1" library="SparkFun-LED" deviceset="LED" device="0603"/>
+<part name="D2" library="SparkFun-LED" deviceset="LED" device="0603"/>
+<part name="R3" library="SparkFun-Resistors" deviceset="300OHM-1/10W-1%(0603)" device="" value="300"/>
+<part name="C2" library="SparkFun-Capacitors" deviceset="4.7UF-6.3V-10%(0603)" device="0603" value="4.7uF"/>
 </parts>
 <sheets>
@@
 <instance part="J2" gate="G$1" x="5.08" y="66.04" rot="R180"/>
 <instance part="F1" gate="G$1" x="2.54" y="45.72"/>
+<instance part="S1" gate="S" x="134.62" y="91.44"/>
+<instance part="D1" gate="G$1" x="27.94" y="83.82"/>
+<instance part="D2" gate="G$1" x="38.1" y="83.82"/>
+<instance part="R3" gate="G$1" x="22.86" y="78.74"/>
+<instance part="C2" gate="G$1" x="55.88" y="86.36" rot="R180"/>
 </instances>
 <busses>
@@
 <wire x1="104.14" y1="38.1" x2="106.68" y2="38.1" width="0.1524" layer="91"/>
 <label x="106.68" y="38.1" size="1.016" layer="95" xref="yes"/>
-</segment>
-<segment>
-<pinref part="U$1" gate="G$1" pin="PB5(ADC12)"/>
-<wire x1="104.14" y1="48.26" x2="106.68" y2="48.26" width="0.1524" layer="91"/>
-<label x="106.68" y="48.26" size="1.016" layer="95" xref="yes"/>
 </segment>
 </net>
@@
 <wire x1="66.04" y1="68.58" x2="66.04" y2="71.12" width="0.1524" layer="91"/>
 <junction x="66.04" y="71.12"/>
+<pinref part="C2" gate="G$1" pin="2"/>
+<wire x1="55.88" y1="88.9" x2="66.04" y2="88.9" width="0.1524" layer="91"/>
 </segment>
 <segment>
@@
 <label x="12.7" y="45.72" size="1.016" layer="95" xref="yes"/>
 </segment>
+<segment>
+<pinref part="D1" gate="G$1" pin="A"/>
+<wire x1="27.94" y1="86.36" x2="27.94" y2="88.9" width="0.1524" layer="91"/>
+<label x="27.94" y="88.9" size="1.016" layer="95" rot="R90" xref="yes"/>
+</segment>
 </net>
 <net name="UCAP" class="0">
@@
 </segment>
 </net>
-<net name="N$26" class="0">
-<segment>
-<pinref part="U$1" gate="G$1" pin="PF7(ADC7)"/>
-<wire x1="104.14" y1="93.98" x2="106.68" y2="93.98" width="0.1524" layer="91"/>
-<label x="106.68" y="93.98" size="1.016" layer="95" xref="yes"/>
-</segment>
-</net>
 <net name="BUTTON" class="0">
 <segment>
@@
 <wire x1="104.14" y1="91.44" x2="106.68" y2="91.44" width="0.1524" layer="91"/>
 <label x="106.68" y="91.44" size="1.016" layer="95" xref="yes"/>
+</segment>
+<segment>
+<pinref part="S1" gate="S" pin="1"/>
+<wire x1="129.54" y1="91.44" x2="127" y2="91.44" width="0.1524" layer="91"/>
+<label x="127" y="91.44" size="1.016" layer="95" rot="R180" xref="yes"/>
 </segment>
 </net>
@@
 <wire x1="7.62" y1="66.04" x2="12.7" y2="66.04" width="0.1524" layer="91"/>
 </segment>
+<segment>
+<pinref part="S1" gate="S" pin="3"/>
+<wire x1="139.7" y1="91.44" x2="142.24" y2="91.44" width="0.1524" layer="91"/>
+<label x="142.24" y="91.44" size="1.016" layer="95" xref="yes"/>
+</segment>
+<segment>
+<pinref part="R3" gate="G$1" pin="1"/>
+<wire x1="15.24" y1="78.74" x2="17.78" y2="78.74" width="0.1524" layer="91"/>
+<label x="15.24" y="78.74" size="1.016" layer="95" rot="R180" xref="yes"/>
+</segment>
+<segment>
+<pinref part="C2" gate="G$1" pin="1"/>
+<wire x1="55.88" y1="81.28" x2="55.88" y2="78.74" width="0.1524" layer="91"/>
+</segment>
 </net>
 <net name="UVCC" class="0">
@@
 </segment>
 </net>
+<net name="CLOCK" class="0">
+<segment>
+<pinref part="U$1" gate="G$1" pin="PB5(ADC12)"/>
+<wire x1="104.14" y1="48.26" x2="106.68" y2="48.26" width="0.1524" layer="91"/>
+<label x="106.68" y="48.26" size="1.016" layer="95" xref="yes"/>
+</segment>
+</net>
+<net name="LGND" class="0">
+<segment>
+<pinref part="D1" gate="G$1" pin="C"/>
+<pinref part="D2" gate="G$1" pin="C"/>
+<wire x1="27.94" y1="78.74" x2="38.1" y2="78.74" width="0.1524" layer="91"/>
+<pinref part="R3" gate="G$1" pin="2"/>
+<junction x="27.94" y="78.74"/>
+</segment>
+</net>
+<net name="LED" class="0">
+<segment>
+<pinref part="D2" gate="G$1" pin="A"/>
+<wire x1="38.1" y1="86.36" x2="38.1" y2="88.9" width="0.1524" layer="91"/>
+<label x="38.1" y="88.9" size="1.016" layer="95" rot="R90" xref="yes"/>
+</segment>
+<segment>
+<pinref part="U$1" gate="G$1" pin="PF7(ADC7)"/>
+<wire x1="104.14" y1="93.98" x2="106.68" y2="93.98" width="0.1524" layer="91"/>
+<label x="106.68" y="93.98" size="1.016" layer="95" xref="yes"/>
+</segment>
+</net>
